File: helicoprion.kicad_sch (KiCad schematic)
At the start: 59 parts, among them J2 TRRS, SW1 SW_SPST, SW10 SW_SPST, SW11 SW_SPST, SW12 SW_SPST, SW13 SW_SPST, SW14 SW_SPST, SW15 SW_SPST, SW16 SW_SPST, SW17 SW_SPST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

Commit message: finish layout
Parts:
- removed D24, D25, D26: 1N4148, various:double_sided_hybrid_sod123_tht, symbol Diode:1N4148
- removed H6, H7: MountingHole, MountingHole:MountingHole_2.2mm_M2, symbol Mechanical:MountingHole
- removed SW24, SW25, SW26, SW8: SW_SPST, keyswitches:Kailh_socket_PG1350_reversible, symbol Switch:SW_SPST
- added D4, D5, D7: 1N4148, Keebio-Parts:Diode-dual, symbol Diode:1N4148
- D1, D10, D11, D12, D13, D14, D15, D16, D17, D18, D19, D2, D20, D21, D22, D23, D3, D6, D9: footprint various:double_sided_hybrid_sod123_tht -> Keebio-Parts:Diode-dual
Connections:
- net tlr is gone; now on net col1: SW6.2 (B), U1.13 (10/B6)
- net GND: no longer SW2.1 (A), SW4.1 (A), SW5.1 (A), SW6.1 (A), SW7.1 (A)
- net col1: now also SW4.2 (B), SW5.2 (B), SW7.2 (B); no longer SW10.2 (B), SW11.2 (B), SW3.2 (B), SW9.2 (B), U1.15 (14/B3)
- net col2: now also SW10.2 (B), SW11.2 (B), SW3.2 (B), SW9.2 (B), U1.14 (16/B2); no longer SW1.2 (B), SW12.2 (B), SW13.2 (B), SW14.2 (B), U1.16 (15/B1)
- net col3: now also SW12.2 (B), SW13.2 (B), SW14.2 (B), SW2.2 (B), U1.15 (14/B3); no longer SW15.2 (B), SW16.2 (B), SW17.2 (B), U1.17 (A0/F7)
- net col4: now also SW1.2 (B), SW15.2 (B), SW16.2 (B), SW17.2 (B), U1.16 (15/B1); no longer SW18.2 (B), SW19.2 (B), SW20.2 (B), U1.18 (A1/F6)
- net col5: now also SW18.2 (B), SW19.2 (B), SW20.2 (B), U1.17 (A0/F7); no longer SW21.2 (B), SW22.2 (B), SW23.2 (B), U1.19 (A2/F5)
- net col6: now also SW21.2 (B), SW22.2 (B), SW23.2 (B), U1.18 (A1/F6); no longer U1.20 (A3/F4)
- net row1: now also D3.1 (K), U1.9 (D7/6); no longer U1.6 (SCL/D0/3)
- net row2: now also U1.10 (E6/7), D4.1 (K); no longer U1.7 (D4/4)
- net row3: now also U1.11 (B4/8), D5.1 (K); no longer U1.8 (C6/5)
- net row4: now also U1.12 (B5/9), D7.1 (K); no longer U1.9 (D7/6)
- net at D2.2 (A): now also SW2.1 (A); no longer SW1.1 (A)
- net at D3.2 (A): now also SW5.1 (A)
- net at D1.2 (A): now also SW1.1 (A)
- removed net tll: SW4.2 (B), U1.14 (16/B2)
- removed net tul: SW5.2 (B), U1.11 (B4/8)
- removed net tum: SW2.2 (B), U1.10 (E6/7)
- removed net tur: SW7.2 (B), U1.12 (B5/9)
- new net: D4.2 (A), SW7.1 (A)
- new net: D7.2 (A), SW4.1 (A)
- new net: D5.2 (A), SW6.1 (A)
- no-connect marks 2 -> 7
Other:
- moved on the sheet: D10, D11, D12, D13, D14, D15, D16, D17, D18, D19, D2, D20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
