File: helicoprion.kicad_pcb (KiCad board)
At the start: 2 copper layers, 151.8 x 125.7 mm, 58 parts, among them J1 TRRS, J2 TRRS, SW1 SW_SPST, SW10 SW_SPST, SW11 SW_SPST, SW12 SW_SPST, SW13 SW_SPST, SW14 SW_SPST, SW15 SW_SPST, SW16 SW_SPST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

Commit message: finish layout
Parts:
- removed D24, D25, D26: 1N4148, various:double_sided_hybrid_sod123_tht
- removed H6, H7: MountingHole, MountingHole:MountingHole_2.2mm_M2
- removed SW24, SW25, SW26, SW8: SW_SPST, keyswitches:Kailh_socket_PG1350_reversible
- added D3: 1N4148, Keebio-Parts:Diode-dual, F.Cu at (165.5, 97.0)
- added D4: 1N4148, Keebio-Parts:Diode-dual, F.Cu at (181.6, 117.8)
- added D5: 1N4148, Keebio-Parts:Diode-dual, F.Cu at (178.6, 113.1)
- added D7: 1N4148, Keebio-Parts:Diode-dual, F.Cu at (166.5, 124.1)
- D1, D10, D11, D12, D13, D14, D15, D16, D17, D18, D19, D2, D20, D21, D22, D23, D6, D9: footprint various:double_sided_hybrid_sod123_tht -> Keebio-Parts:Diode-dual
- moved D15 63.5 mm to (101.8, 39.6)
- moved D16 60.3 mm to (101.9, 56.5)
- moved D20 58.1 mm to (88.6, 82.1), turned to 0 degrees
- moved D23 58.0 mm to (78.3, 88.7), turned to 0 degrees
- moved D17 53.2 mm to (107.0, 74.6), turned to 0 degrees
- moved H4 50.1 mm to (121.6, 83.4)
- moved D19 38.2 mm to (95.0, 64.6), turned to 0 degrees
- moved D22 38.2 mm to (77.1, 71.6), turned to 0 degrees
- moved D14 37.5 mm to (122.8, 79.2)
- moved D12 28.7 mm to (134.6, 49.0), turned to -90 degrees
- moved D2 27.1 mm to (153.8, 108.0), turned to 50 degrees
- moved RSW1 27.1 mm to (173.6, 92.0)
- moved D13 26.0 mm to (134.5, 65.9), turned to -90 degrees
- moved D1 20.4 mm to (128.3, 99.2), turned to -30 degrees
- moved U1 20.0 mm to (169.7, 61.1)
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Connections:
- SW1 pad 1: Net-(D2-A) -> Net-(D1-A)
- SW1 pad 2: col2 -> col4
- SW10 pad 2: col1 -> col2
- SW11 pad 2: col1 -> col2
- SW12 pad 2: col2 -> col3
- SW13 pad 2: col2 -> col3
- SW14 pad 2: col2 -> col3
- SW15 pad 2: col3 -> col4
- SW16 pad 2: col3 -> col4
- SW17 pad 2: col3 -> col4
- SW18 pad 2: col4 -> col5
- SW19 pad 2: col4 -> col5
- SW2 pad 1: GND -> Net-(D2-A)
- SW2 pad 2: tum -> col3
- SW20 pad 2: col4 -> col5
- SW21 pad 2: col5 -> col6
- SW22 pad 2: col5 -> col6
- SW23 pad 2: col5 -> col6
- SW3 pad 2: col1 -> col2
- SW4 pad 1: GND -> Net-(D7-A)
- SW4 pad 2: tll -> col1
- SW5 pad 1: GND -> Net-(D3-A)
- SW5 pad 2: tul -> col1
- SW6 pad 1: GND -> Net-(D5-A)
- SW6 pad 2: tlr -> col1
- SW7 pad 1: GND -> Net-(D4-A)
- SW7 pad 2: tur -> col1
- SW9 pad 2: col1 -> col2
- U1 pad 10: tum -> row2
- U1 pad 11: tul -> row3
- U1 pad 12: tur -> row4
- U1 pad 13: tlr -> col1
- U1 pad 14: tll -> col2
- U1 pad 15: col1 -> col3
- U1 pad 16: col2 -> col4
- U1 pad 17: col3 -> col5
- U1 pad 18: col4 -> col6
- U1 pad 19: col5 -> unconnected-(U1-A2/F5-Pad19)
- U1 pad 20: col6 -> unconnected-(U1-A3/F4-Pad20)
- U1 pad 6: row1 -> unconnected-(U1-SCL/D0/3-Pad6)
- U1 pad 7: row2 -> unconnected-(U1-D4/4-Pad7)
- U1 pad 8: row3 -> unconnected-(U1-C6/5-Pad8)
- U1 pad 9: row4 -> row1
Routing:
- net tlr: track 139.4 -> 0.00 mm, vias 2 -> 0
- net tur: track 132.8 -> 0.00 mm, vias 1 -> 0
- net tll: track 116.5 -> 0.00 mm, vias 2 -> 0
- net tul: track 109.2 -> 0.00 mm, vias 1 -> 0
- net tum: track 95.7 -> 0.00 mm, vias 4 -> 0
- net Net-(D26-A): track 64.4 -> 0.00 mm
- net Net-(D15-A): track 69.0 -> 9.43 mm, vias 1 -> 0
- net Net-(D23-A): track 66.2 -> 10.3 mm
- net Net-(D16-A): track 64.0 -> 9.26 mm, vias 1 -> 0
- net Net-(D20-A): track 65.3 -> 10.7 mm
- net Net-(D17-A): track 65.4 -> 13.3 mm, vias 1 -> 0
- net Net-(D25-A): track 49.9 -> 0.00 mm, vias 1 -> 0
- net GND: track 66.9 -> 17.6 mm, vias 60 -> 2
- net Net-(D22-A): track 58.6 -> 9.36 mm, vias 1 -> 0
- net col4: track 181.4 -> 230.4 mm, vias 4 -> 5
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Other:
- board size 151.8 x 125.7 mm -> 134.5 x 126 mm

Commit message: Add ground vias and gerber
Routing:
- net col1: track 206.0 -> 188.1 mm
- net GND: vias 2 -> 19
- net (no net): vias 0 -> 1
Changed lines of the file:
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@@
     (pad_to_mask_clearance 0)
     (pcbplotparams
-      (layerselection 0x0020000_7ffffffe)
+      (layerselection 0x00010fc_ffffffff)
       (plot_on_all_layers_selection 0x0001000_00000000)
       (disableapertmacros false)
-      (usegerberextensions false)
+      (usegerberextensions true)
       (usegerberattributes true)
-      (usegerberadvancedattributes true)
-      (creategerberjobfile true)
+      (usegerberadvancedattributes false)
+      (creategerberjobfile false)
       (dashed_line_dash_ratio 12.000000)
       (dashed_line_gap_ratio 3.000000)
@@
       (psa4output false)
       (plotreference true)
-      (plotvalue true)
+      (plotvalue false)
       (plotinvisibletext false)
       (sketchpadsonfab false)
-      (subtractmaskfromsilk false)
-      (outputformat 4)
+      (subtractmaskfromsilk true)
+      (outputformat 1)
       (mirror false)
       (drillshape 0)
       (scaleselection 1)
-      (outputdirectory "")
+      (outputdirectory "gerber/")
     )
   )
@@
   (gr_arc (start 98.5 23.5) (mid 98.792893 22.792893) (end 99.5 22.5)
     (stroke (width 0.1) (type default)) (layer "Edge.Cuts"))
+  (via (at 168.79 131.77) (size 0.8) (drill 0.4) (layers "F.Cu" "B.Cu") (net 0))
   (segment (start 159.6548 51.783) (end 159.6548 49.914897) (width 0.25) (layer "F.Cu") (net 1))
   (segment (start 160.449697 49.12) (end 162.1282 49.12) (width 0.25) (layer "F.Cu") (net 1))
@@
   (segment (start 160.8018 52.93) (end 159.6548 51.783) (width 0.25) (layer "F.Cu") (net 1))
   (segment (start 159.6548 49.914897) (end 160.449697 49.12) (width 0.25) (layer "F.Cu") (net 1))
+  (via (at 121.48 46.68) (size 0.8) (drill 0.4) (layers "F.Cu" "B.Cu") (free) (net 1))
+  (via (at 74.99 59.38) (size 0.8) (drill 0.4) (layers "F.Cu" "B.Cu") (free) (net 1))
+  (via (at 86.04 52.76) (size 0.8) (drill 0.4) (layers "F.Cu" "B.Cu") (free) (net 1))
+  (via (at 128.79 79.93) (size 0.8) (drill 0.4) (layers "F.Cu" "B.Cu") (free) (net 1))
+  (via (at 153.64 88.25) (size 0.8) (drill 0.4) (layers "F.Cu" "B.Cu") (free) (net 1))
+  (via (at 110.95 45.74) (size 0.8) (drill 0.4) (layers "F.Cu" "B.Cu") (free) (net 1))
+  (via (at 75.09 76.73) (size 0.8) (drill 0.4) (layers "F.Cu" "B.Cu") (free) (net 1))
+  (via (at 154.83 73.42) (size 0.8) (drill 0.4) (layers "F.Cu" "B.Cu") (free) (net 1))
+  (via (at 174.97 136.21) (size 0.8) (drill 0.4) (layers "F.Cu" "B.Cu") (free) (net 1))
   (via (at 168.14 51.76) (size 0.8) (drill 0.4) (layers "F.Cu" "B.Cu") (free) (net 1))
+  (via (at 154.28 65.53) (size 0.8) (drill 0.4) (layers "F.Cu" "B.Cu") (free) (net 1))
+  (via (at 118.91 76.38) (size 0.8) (drill 0.4) (layers "F.Cu" "B.Cu") (free) (net 1))
+  (via (at 180.22 115.06) (size 0.8) (drill 0.4) (layers "F.Cu" "B.Cu") (free) (net 1))
+  (via (at 104.33 63.3) (size 0.8) (drill 0.4) (layers "F.Cu" "B.Cu") (free) (net 1))
+  (via (at 114.15 73.15) (size 0.8) (drill 0.4) (layers "F.Cu" "B.Cu") (free) (net 1))
+  (via (at 182.83 122.46) (size 0.8) (drill 0.4) (layers "F.Cu" "B.Cu") (free) (net 1))
+  (via (at 130.79 83.71) (size 0.8) (drill 0.4) (layers "F.Cu" "B.Cu") (free) (net 1))
   (via (at 169.99 82.45) (size 0.8) (drill 0.4) (layers "F.Cu" "B.Cu") (free) (net 1))
+  (via (at 161.18 79.94) (size 0.8) (drill 0.4) (layers "F.Cu" "B.Cu") (free) (net 1))
   (segment (start 177.3118 51.66) (end 176.0418 50.39) (width 0.25) (layer "B.Cu") (net 1))
   (segment (start 177.3482 54.2) (end 177.3482 51.66) (width 0.25) (layer "B.Cu") (net 1))
@@
   (segment (start 184.87 132.9) (end 184.87 132.02) (width 0.25) (layer "F.Cu") (net 7))
   (segment (start 170.846401 117.359471) (end 172.976401 117.359471) (width 0.25) (layer "F.Cu") (net 7))
-  (segment (start 176.96136 136.18136) (end 175.79 135.01) (width 0.25) (layer "F.Cu") (net 7))
-  (segment (start 163.22 130.03) (end 166.18 127.07) (width 0.25) (layer "F.Cu") (net 7))
   (segment (start 162.1282 74.52) (end 174.14 74.52) (width 0.25) (layer "F.Cu") (net 7))
-  (segment (start 169.79864 144.71136) (end 176.925 137.585) (width 0.25) (layer "F.Cu") (net 7))
   (segment (start 170.2041 141.4541) (end 170.2041 140.7841) (width 0.25) (layer "F.Cu") (net 7))
   (segment (start 173.49 116.845872) (end 173.49 114.27) (width 0.25) (layer "F.Cu") (net 7))
-  (segment (start 169.579905 144.71136) (end 169.79864 144.71136) (width 0.25) (layer "F.Cu") (net 7))
+  (segment (start 173.34 140.951265) (end 173.34 132.56) (width 0.25) (layer "F.Cu") (net 7))
   (segment (start 180.78 127.93) (end 180.78 124.19) (width 0.25) (layer "F.Cu") (net 7))
   (segment (start 185.55 133.58) (end 184.87 132.9) (width 0.25) (layer "F.Cu") (net 7))
@@
   (segment (start 154.649626 120.549626) (end 154.649626 118.059626) (width 0.25) (layer "F.Cu") (net 7))
   (segment (start 172.976401 117.359471) (end 173.49 116.845872) (width 0.25) (layer "F.Cu") (net 7))
+  (segment (start 173.3 132.52) (end 172.976401 132.196401) (width 0.25) (layer "F.Cu") (net 7))
   (segment (start 160.1 125) (end 157.2 122.1) (width 0.25) (layer "F.Cu") (net 7))
   (segment (start 173.49 114.27) (end 170.45 111.23) (width 0.25) (layer "F.Cu") (net 7))
+  (segment (start 173.34 132.56) (end 173.3 132.52) (width 0.25) (layer "F.Cu") (net 7))
   (segment (start 176.100095 135.320095) (end 175.79 135.01) (width 0.25) (layer "F.Cu") (net 7))
   (segment (start 163.22 130.49) (end 163.22 130.03) (width 0.25) (layer "F.Cu") (net 7))
-  (segment (start 167.98 127.07) (end 173.48 121.57) (width 0.25) (layer "F.Cu") (net 7))
   (segment (start 166.98 108.53) (end 166.98 106.59) (width 0.25) (layer "F.Cu") (net 7))
   (segment (start 165.26 135.84) (end 165.26 132.53) (width 0.25) (layer "F.Cu") (net 7))
+  (segment (start 169.579905 144.71136) (end 173.34 140.951265) (width 0.25) (layer "F.Cu") (net 7))
   (segment (start 170.45 111.23) (end 169.68 111.23) (width 0.25) (layer "F.Cu") (net 7))
   (segment (start 184.389905 136.18136) (end 182.05136 136.18136) (width 0.25) (layer "F.Cu") (net 7))
   (segment (start 181.190095 135.320095) (end 176.100095 135.320095) (width 0.25) (layer "F.Cu") (net 7))
-  (segment (start 166.18 127.07) (end 167.98 127.07) (width 0.25) (layer "F.Cu") (net 7))
   (segment (start 172.976401 132.196401) (end 172.976401 117.359471) (width 0.25) (layer "F.Cu") (net 7))
-  (segment (start 173.48 121.57) (end 178.16 121.57) (width 0.25) (layer "F.Cu") (net 7))
   (segment (start 157.2 122.1) (end 156.2 122.1) (width 0.25) (layer "F.Cu") (net 7))
   (segment (start 180.78 124.19) (end 178.16 121.57) (width 0.25) (layer "F.Cu") (net 7))
   (segment (start 169.579905 144.71136) (end 170.63 143.661265) (width 0.25) (layer "F.Cu") (net 7))
   (segment (start 182.05136 136.18136) (end 181.190095 135.320095) (width 0.25) (layer "F.Cu") (net 7))
-  (segment (start 175.79 135.01) (end 172.976401 132.196401) (width 0.25) (layer "F.Cu") (net 7))
+  (segment (start 169.579905 144.71136) (end 169.79864 144.71136) (width 0.25) (layer "F.Cu") (net 7))
   (segment (start 170.63 141.88) (end 170.2041 141.4541) (width 0.25) (layer "F.Cu") (net 7))
-  (segment (start 176.925 137.585) (end 176.925 136.145) (width 0.25) (layer "F.Cu") (net 7))
   (segment (start 163.9 103.51) (end 163.9 102.96) (width 0.25) (layer "F.Cu") (net 7))
   (segment (start 169.68 111.23) (end 166.98 108.53) (width 0.25) (layer "F.Cu") (net 7))
@@
   (segment (start 170.2041 140.7841) (end 165.26 135.84) (width 0.25) (layer "F.Cu") (net 7))
   (segment (start 165.26 132.53) (end 163.22 130.49) (width 0.25) (layer "F.Cu") (net 7))
+  (segment (start 175.79 135.01) (end 173.3 132.52) (width 0.25) (layer "F.Cu") (net 7))
   (via (at 163.9 102.96) (size 0.8) (drill 0.4) (layers "F.Cu" "B.Cu") (net 7))
   (via (at 151.18 114.59) (size 0.8) (drill 0.4) (layers "F.Cu" "B.Cu") (net 7))
